File: board/calcprop.sch (KiCad schematic (older format))
At the start: 104 parts, among them CON1 SD_Card, P1 BATT, P10 PROG, P2 POWER, P3 EXTBATT, P4 EXTDISPLAY, P5 BACKLIGHT, P6 DISPLAY, P7 FPU, P8 EXTSPI, P9 EXTIO, SW1 KEY, SW10 KEY, SW11 KEY, SW12 KEY, SW13 KEY, SW14 KEY, SW15 KEY, SW16 KEY, SW17 KEY, SW18 KEY, SW19 KEY, SW2 KEY, SW20 KEY, SW21 KEY, SW22 KEY, SW23 KEY, SW24 KEY, SW25 KEY, SW26 KEY, SW27 KEY, SW28 KEY, SW29 KEY, SW3 KEY, SW30 KEY, SW31 KEY, SW32 KEY, SW33 KEY, SW34 KEY, SW35 KEY, SW36 KEY, SW37 KEY, SW38 KEY, SW39 KEY, SW4 KEY, SW40 KEY, SW41 KEY, SW42 KEY, SW43 KEY, SW44 KEY, SW45 KEY, SW46 KEY, SW47 KEY, SW48 KEY, SW5 KEY, SW6 KEY, SW7 KEY, SW8 KEY, SW9 KEY, U1 74LS595, U2 P8X32A, U3 MCP3002, U4 LTC3525-3.3, U5 24LC512, U6 SST25VF080, U7 MCP23S17, U8 23xx1024, U9 23xx1024, Y1 5MHz

Commit message: SPI
Parts:
- added R17, R18, R19, R20, R21, R22: 10K, Resistors_SMD:R_0805, symbol R
Connections:
- net GND: now also R17.2, R18.2, R19.2, R20.2, R21.2, R22.2
- net KEYM_ROW0: now also R22.1
- net KEYM_ROW1: now also R21.1
- net KEYM_ROW2: now also R20.1
- net KEYM_ROW3: now also R19.1
- net KEYM_ROW4: now also R18.1
- net KEYM_ROW5: now also R17.1
Changed lines of the file:
@@
 Connection ~ 3200 7300
 Wire Wire Line
-	3500 6900 3500 10800
-Wire Wire Line
-	3800 6800 3800 10800
-Wire Wire Line
-	4100 6700 4100 10800
-Wire Wire Line
-	4400 6600 4400 10800
-Wire Wire Line
-	4700 6500 4700 10800
+	3500 6400 3500 10800
+Wire Wire Line
+	3800 6400 3800 10800
+Wire Wire Line
+	4100 6400 4100 10800
+Wire Wire Line
+	4400 6400 4400 10800
+Wire Wire Line
+	4700 6400 4700 10800
 Connection ~ 3500 10300
 Connection ~ 3800 10300
@@
 	2400 7000 3200 7000
 Wire Wire Line
-	3200 7000 3200 10800
+	3200 6400 3200 10800
 Wire Wire Line
 	1600 9700 1600 9800
@@
 	1    0    0    -1
 $EndComp
+$Comp
+L R R17
+U 1 1 5853EF74
+P 3200 6250
+F 0 "R17" V 3300 6250 50  0000 C CNN
+F 1 "10K" V 3100 6250 50  0000 C CNN
+F 2 "Resistors_SMD:R_0805" V 3130 6250 50  0001 C CNN
+F 3 "" H 3200 6250 50  0000 C CNN
+	1    3200 6250
+	-1   0    0    1
+$EndComp
+$Comp
+L R R18
+U 1 1 5853F3B1
+P 3500 6250
+F 0 "R18" V 3600 6250 50  0000 C CNN
+F 1 "10K" V 3400 6250 50  0000 C CNN
+F 2 "Resistors_SMD:R_0805" V 3430 6250 50  0001 C CNN
+F 3 "" H 3500 6250 50  0000 C CNN
+	1    3500 6250
+	-1   0    0    1
+$EndComp
+$Comp
+L R R19
+U 1 1 5853F507
+P 3800 6250
+F 0 "R19" V 3900 6250 50  0000 C CNN
+F 1 "10K" V 3700 6250 50  0000 C CNN
+F 2 "Resistors_SMD:R_0805" V 3730 6250 50  0001 C CNN
+F 3 "" H 3800 6250 50  0000 C CNN
+	1    3800 6250
+	-1   0    0    1
+$EndComp
+$Comp
+L R R20
+U 1 1 5853F662
+P 4100 6250
+F 0 "R20" V 4200 6250 50  0000 C CNN
+F 1 "10K" V 4000 6250 50  0000 C CNN
+F 2 "Resistors_SMD:R_0805" V 4030 6250 50  0001 C CNN
+F 3 "" H 4100 6250 50  0000 C CNN
+	1    4100 6250
+	-1   0    0    1
+$EndComp
+$Comp
+L R R21
+U 1 1 5853F7CC
+P 4400 6250
+F 0 "R21" V 4500 6250 50  0000 C CNN
+F 1 "10K" V 4300 6250 50  0000 C CNN
+F 2 "Resistors_SMD:R_0805" V 4330 6250 50  0001 C CNN
+F 3 "" H 4400 6250 50  0000 C CNN
+	1    4400 6250
+	-1   0    0    1
+$EndComp
+$Comp
+L R R22
+U 1 1 58540082
+P 4700 6250
+F 0 "R22" V 4800 6250 50  0000 C CNN
+F 1 "10K" V 4600 6250 50  0000 C CNN
+F 2 "Resistors_SMD:R_0805" V 4630 6250 50  0001 C CNN
+F 3 "" H 4700 6250 50  0000 C CNN
+	1    4700 6250
+	-1   0    0    1
+$EndComp
+Connection ~ 3200 7000
+Connection ~ 3500 6900
+Connection ~ 3800 6800
+Connection ~ 4100 6700
+Connection ~ 4400 6600
+Connection ~ 4700 6500
+$Comp
+L GND #PWR053
+U 1 1 58541375
+P 3200 6000
+F 0 "#PWR053" H 3200 5750 50  0001 C CNN
+F 1 "GND" H 3205 5827 50  0000 C CNN
+F 2 "" H 3200 6000 50  0000 C CNN
+F 3 "" H 3200 6000 50  0000 C CNN
+	1    3200 6000
+	-1   0    0    1
+$EndComp
+Wire Wire Line
+	3200 6100 3200 6000
+Wire Wire Line
+	3200 6050 4700 6050
+Wire Wire Line
+	3500 6050 3500 6100
+Connection ~ 3200 6050
+Wire Wire Line
+	3800 6050 3800 6100
+Connection ~ 3500 6050
+Wire Wire Line
+	4100 6050 4100 6100
+Connection ~ 3800 6050
+Wire Wire Line
+	4400 6050 4400 6100
+Connection ~ 4100 6050
+Wire Wire Line
+	4700 6050 4700 6100
+Connection ~ 4400 6050
 $EndSCHEMATC

Commit message: A bunch of stuff
Parts:
- removed P4: EXTDISPLAY, w_smd_strip:bb02-hp08, symbol CONN_01X07
- removed U2: P8X32A, Housings_QFP:LQFP-44_10x10mm_Pitch0.8mm, symbol P8X32A
- added C13, C18, C19: .1uF, Capacitors_SMD:C_0805, symbol C
- added U2: PROPELLER-QFN, symbol PROPELLER-QFN
- added W1: TEST_BATT, symbol TEST_1P
- added W10: TEST_MBUS_MOSI, symbol TEST_1P
- added W11: TEST_MBUS_SCK, symbol TEST_1P
- added W12: TEST_MBUS_CS0, symbol TEST_1P
- added W13: TEST_MBUS_CS1, symbol TEST_1P
- added W14: TEST_MBUS_CS2, symbol TEST_1P
- added W2: TEST_VCC, symbol TEST_1P
- added W3: TEST_GND, symbol TEST_1P
- added W4: TEST_DBUS_CS, symbol TEST_1P
- added W5: TEST_DBUS_RST, symbol TEST_1P
- added W6: TEST_DBUS_A0, symbol TEST_1P
- added W7: TEST_DBUS_SDA, symbol TEST_1P
- added W8: TEST_DBUS_SCL, symbol TEST_1P
- added W9: TEST_MBUS_MISO, symbol TEST_1P
Connections:
- net COMM_RST: now also U2.7 (RESn)
- net COMM_RX: now also U2.44 (P3)
- net COMM_SCL: now also U2.41 (P0)
- net COMM_SDA: now also U2.42 (P1)
- net COMM_TX: now also U2.43 (P2)
- net DBUS_A0: now also U2.34 (P27), W6.1
- net DBUS_CS: now also U2.36 (P29), W4.1
- net DBUS_RST: now also U2.35 (P28), W5.1
- net DBUS_SCL: now also U2.37 (P30), W8.1
- net DBUS_SDA: now also U2.38 (P31), W7.1
- net GND: now also C13.2, C18.2, C19.2, U2.17 (VSS), U2.27 (VSS), U2.39 (VSS), U2.5 (VSS), U2.6 (BOEn), W3.1
- net KEYM_CLK: now also U2.32 (P25)
- net KEYM_DAT: now also U2.33 (P26)
- net KEYM_LAT: now also U2.31 (P24)
- net KEYM_ROW0: now also U2.26 (P23)
- net KEYM_ROW1: now also U2.25 (P22)
- net KEYM_ROW2: now also U2.24 (P21)
- net KEYM_ROW3: now also U2.23 (P20)
- net KEYM_ROW4: now also U2.2 (P5)
- net KEYM_ROW5: now also U2.1 (P4)
- net MBUS_CS0: now also U2.10 (P9), W12.1
- net MBUS_CS1: now also U2.11 (P10), W13.1
- net MBUS_CS2: now also U2.12 (P11), W14.1
- net MBUS_MISO: now also U2.3 (P6), W9.1
- net MBUS_MOSI: now also U2.4 (P7), W10.1
- net MBUS_SCK: now also U2.9 (P8), W11.1
- net PBUS_CS0: now also U2.16 (P15)
- net PBUS_CS1: now also U2.19 (P16)
- net PBUS_CS2: now also U2.20 (P17)
- net PBUS_CS3: now also U2.21 (P18)
- net PBUS_CS4: now also U2.22 (P19)
- net PBUS_MISO: now also U2.13 (P12)
- net PBUS_MOSI: now also U2.14 (P13)
- net PBUS_SCK: now also U2.15 (P14)
- net VCC: now also C13.1, C18.1, C19.1, U2.18 (VDD), U2.30 (VDD), U2.40 (VDD), U2.8 (VDD), W2.1
- net at Y1.2: now also U2.28 (XI)
- net at Y1.1: now also U2.29 (XO)
- net at C5.1, L1.1, P1.2 (P2)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: now also W1.1
Other:
- moved on the sheet: R13, U6, U8, U9, Y1

Commit message: OK
Parts:
- U2: footprint (none) -> Housings_QFP:LQFP-44_10x10mm_Pitch0.8mm
- W1, W10, W11, W12, W13, W14, W2, W3, W4, W5, W6, W7, W8, W9: footprint (none) -> Measurement_Points:Measurement_Point_Round-SMD-Pad_Small

Commit message: More board
Connections:
- net DBUS_A0: now also U2.33 (P26); no longer U2.34 (P27)
- net DBUS_CS: now also U2.35 (P28); no longer U2.36 (P29)
- net DBUS_RST: now also U2.34 (P27); no longer U2.35 (P28)
- net DBUS_SCL: now also U2.31 (P24); no longer U2.37 (P30)
- net DBUS_SDA: now also U2.32 (P25); no longer U2.38 (P31)
- net KEYM_CLK: now also U2.37 (P30); no longer U2.32 (P25)
- net KEYM_DAT: now also U2.38 (P31); no longer U2.33 (P26)
- net KEYM_LAT: now also U2.36 (P29); no longer U2.31 (P24)
- net KEYM_ROW0: now also U2.1 (P4); no longer U2.26 (P23)
- net KEYM_ROW1: now also U2.2 (P5); no longer U2.25 (P22)
- net KEYM_ROW2: now also U2.3 (P6); no longer U2.24 (P21)
- net KEYM_ROW3: now also U2.4 (P7); no longer U2.23 (P20)
- net KEYM_ROW4: now also U2.9 (P8); no longer U2.2 (P5)
- net KEYM_ROW5: now also U2.10 (P9); no longer U2.1 (P4)
- net MBUS_CS0: now also U2.11 (P10); no longer U2.10 (P9)
- net MBUS_CS1: now also U2.16 (P15); no longer U2.11 (P10)
- net MBUS_CS2: now also U2.15 (P14); no longer U2.12 (P11)
- net MBUS_MISO: now also U2.14 (P13); no longer U2.3 (P6)
- net MBUS_MOSI: now also U2.13 (P12); no longer U2.4 (P7)
- net MBUS_SCK: now also U2.12 (P11); no longer U2.9 (P8)
- net PBUS_CS0: now also U2.22 (P19); no longer U2.16 (P15)
- net PBUS_CS1: now also U2.25 (P22); no longer U2.19 (P16)
- net PBUS_CS2: now also U2.24 (P21); no longer U2.20 (P17)
- net PBUS_CS3: now also U2.26 (P23); no longer U2.21 (P18)
- net PBUS_CS4: now also U2.23 (P20); no longer U2.22 (P19)
- net PBUS_MISO: now also U2.19 (P16); no longer U2.13 (P12)
- net PBUS_MOSI: now also U2.20 (P17); no longer U2.14 (P13)
- net PBUS_SCK: now also U2.21 (P18); no longer U2.15 (P14)
Changed lines of the file:
@@
 	1    0    0    -1
 $EndComp
-Text Label 1150 2100 0    60   ~ 0
+Text Label 2450 4000 1    60   ~ 0
 MBUS_MISO
-Text Label 1150 2200 0    60   ~ 0
+Text Label 2350 4000 1    60   ~ 0
 MBUS_MOSI
-Text Label 1150 2700 0    60   ~ 0
+Text Label 2250 4000 1    60   ~ 0
 MBUS_SCK
-Text Label 1150 2800 0    60   ~ 0
+Text Label 1150 2900 0    60   ~ 0
 MBUS_CS0
-Text Label 1150 2900 0    60   ~ 0
+Text Label 2650 4000 1    60   ~ 0
 MBUS_CS1
-Text Label 2250 4000 1    60   ~ 0
+Text Label 2550 4000 1    60   ~ 0
 MBUS_CS2
-Text Label 2350 4000 1    60   ~ 0
+Text Label 2950 4000 1    60   ~ 0
 PBUS_MISO
-Text Label 2450 4000 1    60   ~ 0
+Text Label 3050 4000 1    60   ~ 0
 PBUS_MOSI
-Text Label 2550 4000 1    60   ~ 0
+Text Label 3150 4000 1    60   ~ 0
 PBUS_SCK
-Text Label 2650 4000 1    60   ~ 0
+Text Label 3250 4000 1    60   ~ 0
 PBUS_CS0
-Text Label 2950 4000 1    60   ~ 0
+Text Label 4350 2700 2    60   ~ 0
 PBUS_CS1
-Text Label 3050 4000 1    60   ~ 0
+Text Label 4350 2800 2    60   ~ 0
 PBUS_CS2
-Text Label 3150 4000 1    60   ~ 0
+Text Label 4350 2600 2    60   ~ 0
 PBUS_CS3
 $Comp
@@
 	1    0    0    -1
 $EndComp
+Text Label 1150 2800 0    60   ~ 0
+KEYM_ROW5
+Text Label 1150 2700 0    60   ~ 0
+KEYM_ROW4
+Text Label 1150 2200 0    60   ~ 0
+KEYM_ROW3
+Text Label 1150 2100 0    60   ~ 0
+KEYM_ROW2
+Text Label 1150 2000 0    60   ~ 0
+KEYM_ROW1
 Text Label 1150 1900 0    60   ~ 0
-KEYM_ROW5
-Text Label 1150 2000 0    60   ~ 0
-KEYM_ROW4
-Text Label 4350 2900 2    60   ~ 0
-KEYM_ROW3
-Text Label 4350 2800 2    60   ~ 0
-KEYM_ROW2
-Text Label 4350 2700 2    60   ~ 0
-KEYM_ROW1
-Text Label 4350 2600 2    60   ~ 0
 KEYM_ROW0
-Text Label 4350 2100 2    60   ~ 0
+Text Label 3050 800  3    60   ~ 0
 KEYM_LAT
-Text Label 4350 2000 2    60   ~ 0
+Text Label 2950 800  3    60   ~ 0
 KEYM_CLK
-Text Label 4350 1900 2    60   ~ 0
+Text Label 2850 800  3    60   ~ 0
 KEYM_DAT
 Text Label 2350 800  3    60   ~ 0
@@
 	-1   0    0    1
 $EndComp
-Text Label 2850 800  3    60   ~ 0
+Text Label 4350 2000 2    60   ~ 0
 DBUS_SDA
-Text Label 2950 800  3    60   ~ 0
+Text Label 4350 2100 2    60   ~ 0
 DBUS_SCL
-Text Label 3250 800  3    60   ~ 0
+Text Label 4350 1900 2    60   ~ 0
 DBUS_A0
-Text Label 3050 800  3    60   ~ 0
+Text Label 3150 800  3    60   ~ 0
 DBUS_CS
 Text Label 10100 3250 0    60   ~ 0
@@
 Text Label 10100 2350 0    60   ~ 0
 DBUS_RST
-Text Label 3150 800  3    60   ~ 0
+Text Label 3250 800  3    60   ~ 0
 DBUS_RST
 Text Label 10700 4500 0    60   ~ 0
@@
 Text Label 10700 5300 0    60   ~ 0
 DBUS_SCL
-Text Label 3250 4000 1    60   ~ 0
+Text Label 4350 2900 2    60   ~ 0
 PBUS_CS4
 Text Label 8850 4800 2    60   ~ 0
@@
 $EndComp
 Wire Wire Line
+	2450 3400 2450 4000
+Wire Wire Line
+	2350 3400 2350 4000
+Wire Wire Line
+	2250 3400 2250 4000
+Wire Wire Line
+	1750 2900 1150 2900
+Wire Wire Line
+	2650 3400 2650 4000
+Wire Wire Line
+	2550 3400 2550 4000
+Wire Wire Line
+	3250 1400 3250 800
+Wire Wire Line
+	3750 1900 4350 1900
+Wire Wire Line
+	2950 3400 2950 4000
+Wire Wire Line
+	3050 3400 3050 4000
+Wire Wire Line
+	3150 3400 3150 4000
+Wire Wire Line
+	3250 3400 3250 4000
+Wire Wire Line
+	3750 2700 4350 2700
+Wire Wire Line
+	3750 2800 4350 2800
+Wire Wire Line
+	3750 2600 4350 2600
+Wire Wire Line
+	3750 2900 4350 2900
+Wire Wire Line
+	2250 800  2250 1400
+Wire Wire Line
+	2350 1400 2350 800
+Wire Wire Line
+	2450 1400 2450 800
+Wire Wire Line
+	2550 1400 2550 800
+Wire Wire Line
+	3750 2000 4350 2000
+Wire Wire Line
+	3750 2100 4350 2100
+Wire Wire Line
+	3150 1400 3150 800
+Wire Wire Line
+	2850 1400 2850 800
+Wire Wire Line
+	3750 2300 4750 2300
+Wire Wire Line
+	3750 2400 4750 2400
+Wire Wire Line
+	2950 1400 2950 800
+Wire Wire Line
+	3050 1400 3050 800
+Wire Wire Line
+	1750 1900 1150 1900
+Wire Wire Line
+	1750 2000 1150 2000
+Wire Wire Line
 	1750 2100 1150 2100
 Wire Wire Line
@@
 	1750 2800 1150 2800
 Wire Wire Line
-	1750 2900 1150 2900
-Wire Wire Line
-	2250 3400 2250 4000
-Wire Wire Line
-	3150 1400 3150 800
-Wire Wire Line
-	3250 1400 3250 800
-Wire Wire Line
-	2350 3400 2350 4000
-Wire Wire Line
-	2450 3400 2450 4000
-Wire Wire Line
-	2550 3400 2550 4000
-Wire Wire Line
-	2650 3400 2650 4000
-Wire Wire Line
-	2950 3400 2950 4000
-Wire Wire Line
-	3050 3400 3050 4000
-Wire Wire Line
-	3150 3400 3150 4000
-Wire Wire Line
-	3250 3400 3250 4000
-Wire Wire Line
-	2250 800  2250 1400
-Wire Wire Line
-	2350 1400 2350 800
-Wire Wire Line
-	2450 1400 2450 800
-Wire Wire Line
-	2550 1400 2550 800
-Wire Wire Line
-	2850 1400 2850 800
-Wire Wire Line
-	2950 1400 2950 800
-Wire Wire Line
-	3050 1400 3050 800
-Wire Wire Line
-	3750 1900 4350 1900
-Wire Wire Line
-	3750 2300 4750 2300
-Wire Wire Line
-	3750 2400 4750 2400
-Wire Wire Line
-	3750 2000 4350 2000
-Wire Wire Line
-	3750 2100 4350 2100
-Wire Wire Line
-	3750 2600 4350 2600
-Wire Wire Line
-	3750 2700 4350 2700
-Wire Wire Line
-	3750 2800 4350 2800
-Wire Wire Line
-	3750 2900 4350 2900
-Wire Wire Line
-	1750 2000 1150 2000
-Wire Wire Line
-	1750 1900 1150 1900
-Wire Wire Line
 	1200 8700 650  8700
