File: board/calcprop.kicad_pcb (KiCad board)
At the start: 2 copper layers, 85.8 x 172.3 mm, 105 parts, among them CON1 SD_Card, P1 BATT, P10 PROG, P2 POWER, P3 EXTBATT, P4 EXTDISPLAY, P5 BACKLIGHT, P6 DISPLAY, P7 FPU, P8 EXTSPI, P9 EXTIO, SW1 KEY, SW10 KEY, SW11 KEY, SW12 KEY, SW13 KEY, SW14 KEY, SW15 KEY, SW16 KEY, SW17 KEY, SW18 KEY, SW19 KEY, SW2 KEY, SW20 KEY, SW21 KEY, SW22 KEY, SW23 KEY, SW24 KEY, SW25 KEY, SW26 KEY, SW27 KEY, SW28 KEY, SW29 KEY, SW3 KEY, SW30 KEY, SW31 KEY, SW32 KEY, SW33 KEY, SW34 KEY, SW35 KEY, SW36 KEY, SW37 KEY, SW38 KEY, SW39 KEY, SW4 KEY, SW40 KEY, SW41 KEY, SW42 KEY, SW43 KEY, SW44 KEY, SW45 KEY, SW46 KEY, SW47 KEY, SW48 KEY, SW5 KEY, SW6 KEY, SW7 KEY, SW8 KEY, SW9 KEY, U1 74LS595, U2 P8X32A, U3 MCP3002, U4 LTC3525-3.3, U5 24LC512, U6 SST25VF080, U7 MCP23S17, U8 23xx1024, U9 23xx1024, Y1 5MHz

Commit message: SPI
Parts:
- added R17: 10K, Resistors_SMD:R_0805, F.Cu at (91.2, 105.7)
- added R18: 10K, Resistors_SMD:R_0805, F.Cu at (78.4, 105.7)
- added R19: 10K, Resistors_SMD:R_0805, F.Cu at (60.7, 105.7)
- added R20: 10K, Resistors_SMD:R_0805, F.Cu at (50.4, 105.7)
- added R21: 10K, Resistors_SMD:R_0805, F.Cu at (36.7, 105.7)
- added R22: 10K, Resistors_SMD:R_0805, F.Cu at (45.7, 91.2)
Routing:
- net GND: track 479.3 -> 636.3 mm, vias 4 -> 13
- net /KEYM_ROW1: track 270.5 -> 275.5 mm
- net /KEYM_ROW5: track 211.4 -> 215.3 mm
- net /KEYM_ROW2: track 290.2 -> 294.1 mm
- net /KEYM_ROW3: track 222.3 -> 225.6 mm
- net /KEYM_ROW4: track 209.4 -> 210.7 mm
Other:
- rule pad_to_mask_clearance: 0.2 -> 0.15

Commit message: OK
Parts:
- removed P4: EXTDISPLAY, w_smd_strip:bb02-hp08
- removed REF***: OSHW-Symbol_8.9x8mm_SilkScreen, Symbols:OSHW-Symbol_8.9x8mm_SilkScreen
- added C13: .1uF, Capacitors_SMD:C_0805, B.Cu at (64.4, 49.0)
- added C18: .1uF, Capacitors_SMD:C_0805, B.Cu at (61.2, 43.8)
- added C19: .1uF, Capacitors_SMD:C_0805, F.Cu at (76.0, 39.2)
- added W1: TEST_BATT, Measurement_Points:Measurement_Point_Round-SMD-Pad_Small, B.Cu at (33.0, 53.9)
- added W10: TEST_MBUS_MOSI, Measurement_Points:Measurement_Point_Round-SMD-Pad_Small, B.Cu at (67.1, 55.8)
- added W11: TEST_MBUS_SCK, Measurement_Points:Measurement_Point_Round-SMD-Pad_Small, B.Cu at (64.8, 55.8)
- added W12: TEST_MBUS_CS0, Measurement_Points:Measurement_Point_Round-SMD-Pad_Small, B.Cu at (55.0, 60.4)
- added W13: TEST_MBUS_CS1, Measurement_Points:Measurement_Point_Round-SMD-Pad_Small, B.Cu at (66.4, 67.4)
- added W14: TEST_MBUS_CS2, Measurement_Points:Measurement_Point_Round-SMD-Pad_Small, B.Cu at (78.8, 62.9)
- added W2: TEST_VCC, Measurement_Points:Measurement_Point_Round-SMD-Pad_Small, B.Cu at (29.9, 74.0)
- added W3: TEST_GND, Measurement_Points:Measurement_Point_Round-SMD-Pad_Small, B.Cu at (34.2, 74.0)
- added W4: TEST_DBUS_CS, Measurement_Points:Measurement_Point_Round-SMD-Pad_Small, B.Cu at (63.4, 21.7)
- added W5: TEST_DBUS_RST, Measurement_Points:Measurement_Point_Round-SMD-Pad_Small, B.Cu at (65.8, 21.7)
- added W6: TEST_DBUS_A0, Measurement_Points:Measurement_Point_Round-SMD-Pad_Small, B.Cu at (69.3, 19.6)
- added W7: TEST_DBUS_SDA, Measurement_Points:Measurement_Point_Round-SMD-Pad_Small, B.Cu at (71.6, 19.6)
- added W8: TEST_DBUS_SCL, Measurement_Points:Measurement_Point_Round-SMD-Pad_Small, B.Cu at (73.9, 19.6)
- added W9: TEST_MBUS_MISO, Measurement_Points:Measurement_Point_Round-SMD-Pad_Small, B.Cu at (78.8, 58.0)
- U2: value P8X32A -> PROPELLER-QFN
- moved P10 9.03 mm to (31.4, 31.2)
- moved R13 5.02 mm to (77.5, 70.4), turned to 270 degrees
- moved C6 4.02 mm to (65.4, 45.6)
- moved C8 4.01 mm to (65.2, 61.5)
- moved R9 3.90 mm to (58.7, 60.4)
- moved C11 3.82 mm to (60.2, 47.2)
- moved R19 3.30 mm to (64.0, 105.7), turned to 0 degrees
- moved L1 2.80 mm to (40.5, 53.5), turned to 180 degrees
- moved U3 2.62 mm to (45.9, 63.1)
- moved U6 2.55 mm to (60.4, 64.4)
- moved P3 2.55 mm to (44.6, 70.2)
- moved C1 2.51 mm to (50.7, 65.8)
- moved P1 2.33 mm to (40.2, 62.9)
- moved C9 2.24 mm to (78.3, 67.4), turned to 0 degrees
- moved C3 2.20 mm to (100.8, 27.1)
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Connections:
- U2 pad 10: GND -> /MBUS_CS0
- U2 pad 11: /COMM_RST -> /MBUS_CS1
- U2 pad 12: VCC -> /MBUS_CS2
- U2 pad 17: /PBUS_CS1 -> GND
- U2 pad 18: /PBUS_CS2 -> VCC
- U2 pad 19: /PBUS_CS3 -> /PBUS_CS1
- U2 pad 20: /PBUS_CS4 -> /PBUS_CS2
- U2 pad 21: /KEYM_ROW3 -> /PBUS_CS3
- U2 pad 22: /KEYM_ROW2 -> /PBUS_CS4
- U2 pad 23: /KEYM_ROW1 -> /KEYM_ROW3
- U2 pad 24: /KEYM_ROW0 -> /KEYM_ROW2
- U2 pad 25: /KEYM_LAT -> /KEYM_ROW1
- U2 pad 26: /KEYM_CLK -> /KEYM_ROW0
- U2 pad 27: /KEYM_DAT -> GND
- U2 pad 28: /DBUS_A0 -> Net-(U2-Pad28)
- U2 pad 29: GND -> Net-(U2-Pad29)
- U2 pad 30: Net-(U2-Pad30) -> VCC
- U2 pad 31: Net-(U2-Pad31) -> /KEYM_LAT
- U2 pad 32: VCC -> /KEYM_CLK
- U2 pad 33: /DBUS_RST -> /KEYM_DAT
- U2 pad 34: /DBUS_CS -> /DBUS_A0
- U2 pad 35: /DBUS_SCL -> /DBUS_RST
- U2 pad 36: /DBUS_SDA -> /DBUS_CS
- U2 pad 37: /COMM_SCL -> /DBUS_SCL
- U2 pad 38: /COMM_SDA -> /DBUS_SDA
- U2 pad 39: /COMM_TX -> GND
- U2 pad 40: /COMM_RX -> VCC
- U2 pad 41: (no net) -> /COMM_SCL
- U2 pad 42: (no net) -> /COMM_SDA
- U2 pad 43: (no net) -> /COMM_TX
- U2 pad 44: (no net) -> /COMM_RX
- U2 pad 5: /MBUS_SCK -> GND
- U2 pad 6: /MBUS_CS0 -> GND
- U2 pad 7: /MBUS_CS1 -> /COMM_RST
- U2 pad 8: /MBUS_CS2 -> VCC
- U2 pad 9: GND -> /MBUS_SCK
- Y1 pad 1: Net-(U2-Pad31) -> Net-(U2-Pad29)
- Y1 pad 2: Net-(U2-Pad30) -> Net-(U2-Pad28)
Routing:
- net GND: track 636.3 -> 0.00 mm, vias 13 -> 0
- net VCC: track 386.4 -> 32.0 mm, vias 9 -> 11
- net /PBUS_MOSI: track 193.0 -> 0.00 mm
- net Net-(SW16-Pad2): track 188.0 -> 0.00 mm, vias 1 -> 0
- net Net-(SW15-Pad2): track 182.4 -> 0.00 mm, vias 1 -> 0
- net Net-(SW14-Pad2): track 176.8 -> 0.00 mm
- net /KEYM_ROW2: track 294.1 -> 141.6 mm, vias 1 -> 0
- net Net-(SW13-Pad2): track 148.8 -> 0.00 mm, vias 1 -> 0
- net /PBUS_MISO: track 143.4 -> 0.00 mm, vias 3 -> 0
- net Net-(SW11-Pad2): track 140.7 -> 0.00 mm
- net Net-(SW12-Pad2): track 135.1 -> 0.00 mm
- net /KEYM_ROW1: track 275.5 -> 141.6 mm, vias 1 -> 0
- net Net-(SW1-Pad2): track 130.6 -> 0.00 mm
- net Net-(SW10-Pad2): track 126.2 -> 0.00 mm, vias 1 -> 0
- net /KEYM_ROW0: track 163.9 -> 44.1 mm, vias 2 -> 0
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- removed copper zone on B.Cu, net GND
- removed copper zone on F.Cu, net GND
Other:
- board size 85.8 x 172.3 mm -> 86.6 x 171.6 mm
- board text added: "Calcular v2 John Lemme Jacob Meyerson"
- board text added: "for real this time i promise"
- board text removed: "CalcLR John Lemme Jacob Meyerson"
- board text removed: "rise and shout it's finished : )"

Commit message: More board
Connections:
- U2 pad 1: /KEYM_ROW5 -> /KEYM_ROW0
- U2 pad 10: /MBUS_CS0 -> /KEYM_ROW5
- U2 pad 11: /MBUS_CS1 -> /MBUS_CS0
- U2 pad 12: /MBUS_CS2 -> /MBUS_SCK
- U2 pad 13: /PBUS_MISO -> /MBUS_MOSI
- U2 pad 14: /PBUS_MOSI -> /MBUS_MISO
- U2 pad 15: /PBUS_SCK -> /MBUS_CS2
- U2 pad 16: /PBUS_CS0 -> /MBUS_CS1
- U2 pad 19: /PBUS_CS1 -> /PBUS_MISO
- U2 pad 2: /KEYM_ROW4 -> /KEYM_ROW1
- U2 pad 20: /PBUS_CS2 -> /PBUS_MOSI
- U2 pad 21: /PBUS_CS3 -> /PBUS_SCK
- U2 pad 22: /PBUS_CS4 -> /PBUS_CS0
- U2 pad 23: /KEYM_ROW3 -> /PBUS_CS4
- U2 pad 24: /KEYM_ROW2 -> /PBUS_CS2
- U2 pad 25: /KEYM_ROW1 -> /PBUS_CS1
- U2 pad 26: /KEYM_ROW0 -> /PBUS_CS3
- U2 pad 3: /MBUS_MISO -> /KEYM_ROW2
- U2 pad 31: /KEYM_LAT -> /DBUS_SCL
- U2 pad 32: /KEYM_CLK -> /DBUS_SDA
- U2 pad 33: /KEYM_DAT -> /DBUS_A0
- U2 pad 34: /DBUS_A0 -> /DBUS_RST
- U2 pad 35: /DBUS_RST -> /DBUS_CS
- U2 pad 36: /DBUS_CS -> /KEYM_LAT
- U2 pad 37: /DBUS_SCL -> /KEYM_CLK
- U2 pad 38: /DBUS_SDA -> /KEYM_DAT
- U2 pad 4: /MBUS_MOSI -> /KEYM_ROW3
- U2 pad 9: /MBUS_SCK -> /KEYM_ROW4
Routing:
- net GND: track 0.00 -> 669.0 mm, vias 0 -> 5
- net VCC: track 32.0 -> 386.2 mm, vias 11 -> 12
- net Net-(SW15-Pad2): track 0.00 -> 204.1 mm
- net Net-(SW16-Pad2): track 0.00 -> 184.6 mm, vias 0 -> 1
- net Net-(SW14-Pad2): track 0.00 -> 171.2 mm
- net Net-(SW11-Pad2): track 0.00 -> 157.5 mm
- net Net-(SW10-Pad2): track 0.00 -> 146.2 mm
- net /PBUS_SCK: track 0.00 -> 143.7 mm, vias 0 -> 1
- net Net-(SW13-Pad2): track 0.00 -> 142.7 mm
- net Net-(SW12-Pad2): track 0.00 -> 137.9 mm
- net Net-(SW1-Pad2): track 0.00 -> 135.1 mm
- net /PBUS_MISO: track 0.00 -> 127.0 mm, vias 0 -> 3
- net /PBUS_MOSI: track 0.00 -> 123.7 mm, vias 0 -> 2
- net /KEYM_ROW0: track 44.1 -> 149.0 mm, vias 0 -> 1
- net /DBUS_BCKL: track 0.00 -> 76.4 mm
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
Commit message: New board complete
Routing:
- added copper zone on B.Cu, net GND
- added copper zone on F.Cu, net GND
Changed lines of the file:
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@@
-(kicad_pcb (version 20160815) (host pcbnew no-vcs-found-7475~57~ubuntu16.10.1)
+(kicad_pcb (version 20160815) (host pcbnew no-vcs-found-7415~56~ubuntu16.10.1)
   (general
     (links 418)
     (no_connects 0)
-    (area 20.524999 16.6425 109.45 189.875001)
+    (area 20.624999 18.124999 107.375001 189.875001)
     (thickness 1.6)
-    (drawings 12)
+    (drawings 23)
     (tracks 1583)
     (zones 0)
@@
     (tags "capacitor 0805")
     (attr smd)
-    (fp_text reference C2 (at 0 1.6 270) (layer B.SilkS)
+    (fp_text reference C2 (at 2.8 0.1 270) (layer B.SilkS)
       (effects (font (size 1 1) (thickness 0.15)) (justify mirror))
     )
@@
     (tags "capacitor 0805")
     (attr smd)
-    (fp_text reference C8 (at 0 1.7 90) (layer B.SilkS)
+    (fp_text reference C8 (at -3.8 0.65 90) (layer B.SilkS)
       (effects (font (size 1 1) (thickness 0.15)) (justify mirror))
     )
@@
     (tags "capacitor 0805")
     (attr smd)
-    (fp_text reference C9 (at 0 1.6) (layer B.SilkS)
+    (fp_text reference C9 (at 1.25 1.8) (layer B.SilkS)
       (effects (font (size 1 1) (thickness 0.15)) (justify mirror))
     )
@@
     (tags "Mesurement Point Round SMD Pad 1.5mm")
     (attr virtual)
-    (fp_text reference W6 (at 0 2) (layer B.SilkS)
+    (fp_text reference W6 (at 9.15 2.7) (layer B.SilkS)
       (effects (font (size 1 1) (thickness 0.15)) (justify mirror))
     )
@@
     (tags "Mesurement Point Round SMD Pad 1.5mm")
     (attr virtual)
-    (fp_text reference W7 (at 0 2) (layer B.SilkS)
+    (fp_text reference W7 (at 5.75 1.35) (layer B.SilkS)
       (effects (font (size 1 1) (thickness 0.15)) (justify mirror))
     )
@@
     (tags "Mesurement Point Round SMD Pad 1.5mm")
     (attr virtual)
-    (fp_text reference W8 (at 0 2) (layer B.SilkS)
+    (fp_text reference W8 (at 2.35 0) (layer B.SilkS)
       (effects (font (size 1 1) (thickness 0.15)) (justify mirror))
     )
@@
     (tags "Mesurement Point Round SMD Pad 1.5mm")
     (attr virtual)
-    (fp_text reference W10 (at 0 2) (layer B.SilkS)
+    (fp_text reference W10 (at 0.5 2.05) (layer B.SilkS)
       (effects (font (size 1 1) (thickness 0.15)) (justify mirror))
     )
@@
     (tags "Mesurement Point Round SMD Pad 1.5mm")
     (attr virtual)
-    (fp_text reference W11 (at 0 2) (layer B.SilkS)
+    (fp_text reference W11 (at -0.6 2.05) (layer B.SilkS)
       (effects (font (size 1 1) (thickness 0.15)) (justify mirror))
     )
@@
       (net 56 /MBUS_CS2))
   )
+  (gr_circle (center 25.25 43.05) (end 25.2 43.7) (layer F.SilkS) (width 0.2))
+  (gr_circle (center 44.6 73.1) (end 44.95 73.7) (layer F.SilkS) (width 0.2))
+  (gr_circle (center 37.65 74.85) (end 38.2 75.25) (layer F.SilkS) (width 0.2))
+  (gr_circle (center 49.55 60.2) (end 49.5 60.85) (layer F.SilkS) (width 0.2))
+  (gr_circle (center 38.4 59.05) (end 38.8 59.4) (layer F.SilkS) (width 0.2))
+  (gr_circle (center 82.1 27.3) (end 82.75 27.8) (layer F.SilkS) (width 0.2))
+  (gr_circle (center 69.6 65.65) (end 69.55 66.3) (layer F.SilkS) (width 0.2))
+  (gr_circle (center 75.2 63.2) (end 75.15 63.85) (layer F.SilkS) (width 0.2))
+  (gr_circle (center 57.65 60.85) (end 57.6 61.5) (layer F.SilkS) (width 0.2))
+  (gr_circle (center 56.7 52.15) (end 57.25 52.6) (layer F.SilkS) (width 0.2))
+  (gr_circle (center 55.9 83.7) (end 56.6 84.05) (layer F.SilkS) (width 0.2))
   (gr_line (start 99.1 83) (end 99.1 189.8) (angle 90) (layer Edge.Cuts) (width 0.15))
   (gr_line (start 28.9 83) (end 28.9 189.8) (angle 90) (layer Edge.Cuts) (width 0.15))
@@
   (segment (start 58.0506 34.3) (end 62.8 39.0494) (width 0.25) (layer F.Cu) (net 90))
   (segment (start 50.1489 34.3) (end 58.0506 34.3) (width 0.25) (layer F.Cu) (net 90))
+  (zone (net 2) (net_name GND) (layer F.Cu) (hatch edge 0.508)
+    (connect_pads (clearance 0.508))
+    (min_thickness 0.254)
+    (fill yes (arc_segments 16) (thermal_gap 0.508) (thermal_bridge_width 0.508))
+    (polygon
+      (pts
+        (xy 107.2 74.75) (xy 99 82.95) (xy 99 189.7) (xy 29 189.7) (xy 29 82.95)
+        (xy 20.8 74.75) (xy 20.8 18.3) (xy 107.2 18.3)
+      )
+    )
+  )
+  (zone (net 2) (net_name GND) (layer B.Cu) (hatch edge 0.508)
+    (connect_pads (clearance 0.508))
+    (min_thickness 0.254)
+    (fill yes (arc_segments 16) (thermal_gap 0.508) (thermal_bridge_width 0.508))
+    (polygon
+      (pts
+        (xy 107.2 74.75) (xy 99 82.95) (xy 99 189.7) (xy 29 189.7) (xy 29 82.95)
+        (xy 20.8 74.75) (xy 20.8 18.3) (xy 107.2 18.3)
+      )
+    )
+  )
 )

Commit message: First draft of case
Parts:
- moved CON1 0.21 mm to (109.2, 31.4)
